Commit message: fix error time out position mode

File: ros2_canopen/canopen_tests/urdf/robot_controller/robot_controller.ros2_control.xacro (robot description, xacro)
@@ -20,8 +20,8 @@
                 <state_interface name="position" />
             </joint>
-            <joint name="${prefix}joint2">
+            <!-- <joint name="${prefix}joint2">
                 <param name="device_name">joint_2</param>
                 <state_interface name="position" />
-            </joint>
+            </joint> -->
         </ros2_control>
     </xacro:macro>
